File: PSU.sch (KiCad schematic (older format))
At the start: 66 parts, among them Q1 NPN, Q2 PNP, Q3 BD241A, T1 AMGIS_L01, U2 LM317T

Commit message: Started work on changing the PSU to fully complementary.
Parts:
- removed C?: 47u, symbol CP1
- removed C?: 10u, symbol CP1
- removed C? (x3): 100n, symbol C
- removed C?: 100u, symbol CP1
- removed C?: 47n, symbol C
- removed D2: BRIDGE_SML, symbol BRIDGE_SML
- removed D6: DIODE, ~, symbol DIODE
- removed D?: ZENER, symbol ZENER
- removed D?: DIODESCH, symbol DIODESCH
- removed Q1: NPN, ~, symbol NPN
- removed Q2: PNP, ~, symbol PNP
- removed Q?: BD241A, TO-220, symbol BD241A
- removed R7, R8: 1.2k, symbol R
- removed R?: 47, symbol R
- removed R?: 4.99k, ~, symbol R
- removed R?: 10k, ~, symbol R
- removed R?: 3.32k, ~, symbol R
- removed R?: 1k, symbol R
- removed U?: LM317T, TO-220, symbol LM317T
- removed U?: OPA209-SOT23, symbol OPA209-SOT23
- removed U?: REF02, symbol REF02
- removed U?: SCR_SML, symbol SCR_SML
- added C? (x2): 100n, symbol C
- added C?: 10u, symbol CP1
- added C?: 47u, symbol CP1
- added C?: 100u, symbol CP1
- added C?: 47n, symbol C
- added D?: ZENER, symbol ZENER
- added D?: DIODESCH, symbol DIODESCH
- added R?: 4.99k, ~, symbol R
- added R?: 3.32k, ~, symbol R
- added R?: 47, symbol R
- added R?: 10k, ~, symbol R
- added R?: 1k, symbol R
- added U?: LM337T, TO-220, symbol LM337T
- added U?: OPA209-SOT23, symbol OPA209-SOT23
- added U?: SCR_SML, symbol SCR_SML
Connections:
- wire segments 143 -> 104
- no-connect marks 4 -> 2
Other:
- moved on the sheet: C1, C12, C14, C3, C6, C?, D1, D4, D?, Q3, R11, R12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
