File: kicad/usb_bridge/test_i2s_gen_cpld/test_i2s_gen.sch (KiCad schematic (older format))
At the start: 82 parts, among them J1 Conn_01x02_Male, J2 Conn_02x05_Odd_Even, J3 Conn_01x02_Male, U1 SIT2001B, U2 AMS1117-3.3, U3 AMS1117-1.8, U4 5M40ZE64C5N

Commit message: I2S test generator refinements
Parts:
- removed C1: 10u, Capacitor_SMD:C_0805_2012Metric, symbol Device:C
- removed H1, H2, H3, H4: MountingHole, MountingHole:MountingHole_2.2mm_M2, symbol Mechanical:MountingHole
- removed R3, R4: R, Resistor_SMD:R_0603_1608Metric, symbol Device:R
- removed TP1, TP10, TP11, TP12, TP13, TP14, TP15, TP16, TP17, TP18, TP19, TP2, TP20, TP21, TP22, TP23, TP24, TP25, TP26, TP27, TP28, TP29, TP3, TP30, TP31, TP32, TP33, TP34, TP35, TP36, TP37, TP38, TP39, TP4, TP40, TP41, TP42, TP43, TP44, TP45, TP46, TP47, TP48, TP49, TP5, TP50, TP51, TP52, TP53, TP54, TP6, TP7, TP8, TP9: ~, Connector_PinHeader_2.54mm:PinHeader_1x01_P2.54mm_Vertical, symbol Connector:TestPoint_Small
- added J4: Conn_01x04_Male, Connector_PinHeader_2.54mm:PinHeader_1x04_P2.54mm_Vertical, symbol Connector:Conn_01x04_Male
- C10: renamed from C8; symbol Device:C -> Device:C_Small
- C11: renamed from C10; symbol Device:C -> Device:C_Small
- C6: renamed from C5; symbol Device:C -> Device:C_Small
- C7: symbol Device:C -> Device:C_Small
- C8: renamed from C11; symbol Device:C -> Device:C_Small
- C9: renamed from C12; symbol Device:C -> Device:C_Small
- J2: DigiKey (none) -> ED1543-ND
- S1: footprint digikey-footprints:Switch_Tactile_THT_6x6mm -> project_footprints:Switch_Tactile_THT_6x6mm; Category Switches -> (none); DK_Datasheet_Link https://www.te.com/commerce/DocumentDelivery/DDEController?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 -> (none); DK_Detail_Page /product-detail/en/te-connectivity-alcoswitch-switches/1825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 -> (none); Description SWITCH TACTILE SPST-NO 0.05A 24V -> (none); Digi-Key_PN 450-1650-ND -> (none); DigiKey (none) -> 450-1650-ND; Family Tactile Switches -> (none); MPN 1825910-6 -> (none); Manufacturer TE Connectivity ALCOSWITCH Switches -> (none); Status Active -> (none)
- U2: DigiKey (none) -> AZ1117IH-3.3TRG1DICT-ND
- U3: DigiKey (none) -> AZ1117EH-1.8TRG1DICT-ND
- U4: DigiKey (none) -> 544-2717-ND
- renumbered C4 to C1, C6 to C4, C9 to C5
Connections:
- net +1V8: now also J2.4 (Pin_4)
- net +3V3: now also U4.5
- net GNDD: now also J4.1 (Pin_1)
- net Vcc: now reaches C2.1, J1.1 (Pin_1), U2.3 (VI)
- net ~RESET: now reaches U4.4
- net ~RESET: now also C3.1, R1.1, R2.2, S1.2
- net LRCK: now reaches U4.51
- net LRCK: now also J4.3 (Pin_3)
- net DATA: now reaches U4.52
- net DATA: now also J4.2 (Pin_2)
- net BCK: now reaches U4.53
- net BCK: now also J4.4 (Pin_4)
- net CLK12: now reaches U4.7
- net CLK12: now also J3.2 (Pin_2)
- net at U4.9: no longer J3.1 (Pin_1)
- net CLK2: no longer names the net of U1.5 (Out)
- net CLK2: now also J3.1 (Pin_1); no longer J3.2 (Pin_2)
- now unconnected: S1.1
- no-connect marks 3 -> 52
Other:
- note added: "12.288 MHz"
- note added: "Disconnect CLK when programming"
- moved on the sheet: C1, C10, C11, C2, C3, C4, C5, C6, C7, C8, C9, J1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
